File: eagle projects/ADCS Actuator Board/ActuatorBoard.brd (EAGLE design)
At the start: 91 x 91 mm, 228 parts, among them J11 TE_1-84953-1, J2 TE_1-84953-1, J4 TE_1-84953-1, J5 TE-1734829-3, U1 SIP2100DY-T1-GE3, U10 LM2917MX/NOPB, U12 TSV991AILT, U13 LM2917MX/NOPB, U14 ADS7841E_2K5, U16 DRV10970_MOTOR_DRIVERDRV10970, U17 LM2917MX/NOPB, U19 TSV991AILT, U2 SIP2100DY-T1-GE3, U20 ADS7841E_2K5, U3 SIP2100DY-T1-GE3, U6 DRV10970_MOTOR_DRIVERDRV10970, U7 DRV10970_MOTOR_DRIVERDRV10970, U8 TSV991AILT, U9 ADS7841E_2K5

Commit message: Updated Actuator board BOM and populated necessary resistors on Z+ board
Parts:
- R22, R42, R88: value DNP -> 470R
Changed lines of the file:
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@@
 <attribute name="VALUE" x="24.4475" y="46.6725" size="1.27" layer="27" rot="R90"/>
 </element>
-<element name="R22" library="rcl" library_urn="urn:adsk.eagle:library:334" package="R0805" package3d_urn="urn:adsk.eagle:package:23553/2" value="DNP" x="18.415" y="48.26" smashed="yes" rot="MR90">
+<element name="R22" library="rcl" library_urn="urn:adsk.eagle:library:334" package="R0805" package3d_urn="urn:adsk.eagle:package:23553/2" value="470R" x="18.415" y="48.26" smashed="yes" rot="MR90">
 <attribute name="NAME" x="19.05" y="46.0375" size="1.016" layer="26" rot="MR270"/>
 <attribute name="POPULARITY" value="85" x="18.415" y="48.26" size="1.778" layer="28" rot="MR90" display="off"/>
@@
 <attribute name="VALUE" x="24.4475" y="59.3725" size="1.27" layer="27" rot="R90"/>
 </element>
-<element name="R42" library="rcl" library_urn="urn:adsk.eagle:library:334" package="R0805" package3d_urn="urn:adsk.eagle:package:23553/2" value="DNP" x="18.415" y="60.96" smashed="yes" rot="MR90">
+<element name="R42" library="rcl" library_urn="urn:adsk.eagle:library:334" package="R0805" package3d_urn="urn:adsk.eagle:package:23553/2" value="470R" x="18.415" y="60.96" smashed="yes" rot="MR90">
 <attribute name="NAME" x="18.7325" y="59.055" size="1.016" layer="26" rot="MR270"/>
 <attribute name="POPULARITY" value="85" x="18.415" y="60.96" size="1.778" layer="28" rot="MR90" display="off"/>
@@
 <attribute name="VALUE" x="24.4475" y="72.0725" size="1.27" layer="27" rot="R90"/>
 </element>
-<element name="R88" library="rcl" library_urn="urn:adsk.eagle:library:334" package="R0805" package3d_urn="urn:adsk.eagle:package:23553/2" value="DNP" x="18.415" y="73.66" smashed="yes" rot="MR90">
+<element name="R88" library="rcl" library_urn="urn:adsk.eagle:library:334" package="R0805" package3d_urn="urn:adsk.eagle:package:23553/2" value="470R" x="18.415" y="73.66" smashed="yes" rot="MR90">
 <attribute name="NAME" x="19.05" y="71.755" size="1.016" layer="26" rot="MR270"/>
 <attribute name="POPULARITY" value="85" x="18.415" y="73.66" size="1.778" layer="28" rot="MR90" display="off"/>
